File: SmokeSensor/SmokeSensor/ESP32.kicad_sch (KiCad schematic)
At the start: 12 parts, among them SW1 RESET, SW2 BOOT, U6 ESP32-WROOM-32E

Commit message: layout 2-layers done!
Changed lines of the file:
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@@
+		)
+	)
+	(text_box "ESP32              LCD ILI9225\n------             -------------\nGPIO23 (MOSI) ---> SDA\nGPIO18 (SCK)  ---> SCK\nGPIO19 (MISO) ---> MISO (SD)\n\nGPIO5         ---> CS (LCD)\nGPIO4         ---> CS (SD)\n\nGPIO16        ---> DC (RS)   \nGPIO17        ---> RESET     \n\n3.3V          ---> VCC\nGND           ---> GND"
+		(exclude_from_sim no)
+		(at 222.25 72.39 0)
+		(size 44.45 34.29)
+		(margins 0.9525 0.9525 0.9525 0.9525)
+		(stroke
+			(width 0)
+			(type solid)
+		)
+		(fill
+			(type none)
+		)
+		(effects
+			(font
+				(size 1.27 1.27)
+			)
+			(justify left top)
 		)
 	)
@@
 		(pts
 			(xy 181.61 105.41) (xy 193.04 105.41)
+		)
+		(stroke
+			(width 0)
+			(type default)
+		)
+	)
+	(wire
+		(pts
+			(xy 111.76 60.96) (xy 119.38 60.96)
 		)
 		(stroke
@@
 		)
 	)
+	(hierarchical_label "+3.3V"
+		(shape input)
+		(at 111.76 60.96 180)
+		(effects
+			(font
+				(size 1.27 1.27)
+			)
+			(justify right)
+		)
+	)
