File: SmokeSensor/SmokeSensor/LCD.kicad_sch (KiCad schematic)
At the start: 2 parts, among them J3 Conn_01x11, J4 Conn_01x04

Commit message: layout 2-layers done!
Connections:
- net +3.3V: now also J3.11 (Pin_11); no longer J3.1 (Pin_1)
- net CS_LCD: now also J3.1 (Pin_1); no longer J3.11 (Pin_11)
- net DC(RS): now also J3.3 (Pin_3); no longer J3.9 (Pin_9)
- net GND: now also J3.10 (Pin_10), J3.9 (Pin_9); no longer J3.2 (Pin_2), J3.3 (Pin_3)
- net MISO: no longer J3.8 (Pin_8), J4.3 (Pin_3)
- net RST: now also J3.2 (Pin_2); no longer J3.10 (Pin_10)
- net SCK: now also J3.5 (Pin_5); no longer J3.7 (Pin_7)
- net MOSI: now reaches J3.4 (Pin_4)
- net MOSI: now also J4.3 (Pin_3)
Other:
- moved on the sheet: J3
Changed lines of the file:
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@@
+		(color 0 0 0 0)
+	)
+	(junction
+		(at 119.38 128.27)
+		(diameter 0)
 		(color 0 0 0 0)
 	)
@@
 	(wire
 		(pts
+			(xy 119.38 128.27) (xy 123.19 128.27)
+		)
+		(stroke
+			(width 0)
+			(type default)
+		)
+	)
+	(wire
+		(pts
 			(xy 116.84 107.95) (xy 125.73 107.95)
 		)
@@
 	(wire
 		(pts
+			(xy 119.38 133.35) (xy 119.38 128.27)
+		)
+		(stroke
+			(width 0)
+			(type default)
+		)
+	)
+	(wire
+		(pts
 			(xy 119.38 123.19) (xy 119.38 125.73)
 		)
@@
 	(wire
 		(pts
-			(xy 116.84 128.27) (xy 123.19 128.27)
+			(xy 116.84 128.27) (xy 119.38 128.27)
 		)
 		(stroke
@@
 	(wire
 		(pts
-			(xy 172.72 120.65) (xy 180.34 120.65)
+			(xy 115.57 133.35) (xy 119.38 133.35)
+		)
+		(stroke
+			(width 0)
+			(type default)
+		)
+	)
+	(wire
+		(pts
+			(xy 172.72 120.65) (xy 181.61 120.65)
 		)
 		(stroke
@@
 	)
 	(label "MOSI"
-		(at 180.34 115.57 180)
+		(at 181.61 115.57 180)
 		(effects
 			(font
@@
 		)
 	)
+	(hierarchical_label "+3.3V"
+		(shape input)
+		(at 115.57 133.35 180)
+		(effects
+			(font
+				(size 1.27 1.27)
+			)
+			(justify right)
+		)
+	)
 	(hierarchical_label "MISO"
 		(shape input)
-		(at 181.61 115.57 0)
+		(at 181.61 120.65 0)
 		(effects
 			(font
@@
 	(symbol
 		(lib_id "Connector_Generic:Conn_01x11")
-		(at 111.76 115.57 180)
+		(at 111.76 115.57 0)
+		(mirror y)
 		(unit 1)
 		(exclude_from_sim no)
@@
 		(dnp no)
 		(property "Reference" "J3"
-			(at 109.22 116.8401 0)
+			(at 109.22 114.2999 0)
 			(effects
 				(font
@@
 		)
 		(property "Value" "Conn_01x11"
-			(at 109.22 114.3001 0)
-			(effects
-				(font
+			(at 109.22 116.8399 0)
+			(effects
+				(font
