File: SmokeSensor/SmokeSensor/POWER.kicad_sch (KiCad schematic)
At the start: 19 parts, among them U1 MT3608, U2 TP4056-42-ESOP8, U3 MCP1700x-330xxMB

Commit message: layout 2-layers done!
Parts:
- added J5: Pin lithium, Connector_JST:JST_PH_S2B-PH-K_1x02_P2.00mm_Horizontal, symbol Connector:Conn_01x02_Pin
- added J6: Switch, Connector_PinHeader_2.54mm:PinHeader_1x03_P2.54mm_Vertical, symbol Connector:Conn_01x03_Pin
- L1: value 22uH -> 22uH/2A
- R3: value 1k2 -> 100k
- R4: value 1k2 -> 2k2
Connections:
- net GND: now also J5.2 (Pin_2)
- net VBATT/PWR: now reaches C1.1, L1.1, U1.4 (EN), U1.5 (IN)
- net VBATT/PWR: now also J6.3 (Pin_3)
- net VBATT: now reaches C5.1, U2.5 (BAT)
- net VBATT: now also J5.1 (Pin_1), J6.2 (Pin_2)
- no-connect marks 1 -> 2
Other:
- moved on the sheet: C1, C2, C3, C4, C5, C6, C7, D1, D2, D3, L1, R1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
