File: SmokeSensor/SmokeSensor/Sensors.kicad_sch (KiCad schematic)
At the start: 6 parts, among them J2 Conn_01x05_Pin, U5 SHT31-DIS

Commit message: layout 2-layers done!
Changed lines of the file:
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@@
+	(wire
+		(pts
+			(xy 82.55 86.36) (xy 87.63 86.36)
+		)
+		(stroke
+			(width 0)
+			(type default)
+		)
+	)
 	(wire
 		(pts
@@
 		)
 	)
+	(hierarchical_label "+3.3V"
+		(shape input)
+		(at 82.55 86.36 180)
+		(effects
+			(font
+				(size 1.27 1.27)
+			)
+			(justify right)
+		)
+	)
