File: SmokeSensor/SmokeSensor/USB_UART.kicad_sch (KiCad schematic)
At the start: 14 parts, among them J1 USB_C_Receptacle_USB2.0_16P, Q1 SS8050, Q2 SS8050, U4 CH340C

Commit message: layout 2-layers done!
Changed lines of the file:
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@@
 	(paper "A4")
+	(junction
+		(at 158.75 74.93)
+		(diameter 0)
+		(color 0 0 0 0)
+	)
 	(junction
 		(at 90.17 77.47)
@@
 	(wire
 		(pts
+			(xy 158.75 74.93) (xy 158.75 80.01)
+		)
+		(stroke
+			(width 0)
+			(type default)
+		)
+	)
+	(wire
+		(pts
 			(xy 115.57 97.79) (xy 129.54 97.79)
 		)
@@
 	(wire
 		(pts
-			(xy 158.75 71.12) (xy 158.75 80.01)
+			(xy 158.75 71.12) (xy 158.75 74.93)
 		)
 		(stroke
@@
 	(wire
 		(pts
+			(xy 153.67 74.93) (xy 158.75 74.93)
+		)
+		(stroke
+			(width 0)
+			(type default)
+		)
+	)
+	(wire
+		(pts
 			(xy 71.12 115.57) (xy 71.12 121.92)
 		)
@@
 		(pts
 			(xy 124.46 92.71) (xy 88.9 92.71)
+		)
+		(stroke
+			(width 0)
+			(type default)
+		)
+	)
+	(wire
+		(pts
+			(xy 119.38 77.47) (xy 124.46 77.47)
 		)
 		(stroke
@@
 		)
 	)
+	(hierarchical_label "+3.3V"
+		(shape input)
+		(at 153.67 74.93 180)
+		(effects
+			(font
+				(size 1.27 1.27)
+			)
+			(justify right)
+		)
+	)
+	(hierarchical_label "+5V"
+		(shape input)
+		(at 124.46 77.47 0)
+		(effects
+			(font
+				(size 1.27 1.27)
+			)
+			(justify left)
+		)
+	)
