File: RTC_PUMP12V5A/RTC_PUMP12V5A.kicad_sch (KiCad schematic)
At the start: 66 parts, among them J1 12VDC_IN, J2 USB_C_Receptacle_USB2.0_16P, J3 Pump, J4 OLED SPI, J5 UART, J6 Conn_01x06_Socket, Q1 AO4407A, Q2 IRLR7843, SW1 SW_Push, SW2 SW_Push, U1 LM1117MP-3.3, U2 TPS5430DDA, U3 ESP32-C3-WROOM-02, U4 USBLC6-2SC6, U5 DS3231M

Commit message: layout completed RTC PUMP12V & push HBrigde project
Parts:
- added TP1, TP2: TestPoint, Connector_Pin:Pin_D1.0mm_L10.0mm, symbol Connector:TestPoint
Connections:
- net +12V: now also J3.2 (Pin_2); no longer J3.1 (Pin_1)
- net +3.3V: now also TP2.1
- net 5V: now also TP1.1
- net EN: no longer U2.5 (EN)
- net IO0: now also J6.4 (Pin_4), R16.1, U5.15 (SDA)
- net IO1: now also J6.3 (Pin_3), R15.1, U5.16 (SCL)
- net IO2: no longer J4.7 (Pin_7)
- net IO5: now also J4.6 (Pin_6)
- net IO8: no longer J6.4 (Pin_4), R16.1, U5.15 (SDA)
- net IO9: no longer J6.3 (Pin_3), R15.1, U5.16 (SCL)
- net PUMP: now also U3.10 (IO10); no longer U3.3 (IO4)
- net at D6.2 (A), Q2.2 (D): now also J3.1 (Pin_1); no longer J3.2 (Pin_2)
- removed net IO10: J4.6 (Pin_6), U3.10 (IO10)
- new net EN_PWR: U2.5 (EN)
- new net IO4: J4.7 (Pin_7), U3.3 (IO4)
- no-connect marks 14 -> 11
Other:
- moved on the sheet: J3
