File: HBridge_1Motor/HBridge_1Motor.kicad_sch (KiCad schematic)
At the start: 88 parts, among them IC1 GP1S093HCZ0F, IC2 GP1S093HCZ0F, IC3 GP1S093HCZ0F, IC4 GP1S093HCZ0F, IC5 LM393DR, IC6 MCP6002-I_SN, J1 +24V_Vin, J2 Conn_01x04_Pin, Q1 IRF3205SPBF, Q2 IRF3205SPBF, Q3 IRF3205SPBF, Q4 IRF3205SPBF, Q5 IRF3205SPBF, U1 AMS1117-5.0, U2 XL4015, U3 4001, U4 IR2104, U5 IR2104, U6 6N137, U7 PC817

Commit message: edit HBridge, RTC_Pump, SmokeSensor skillscreen layers
Connections:
- no-connect marks 7 -> 8
Changed lines of the file:
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@@
+	)
+	(no_connect
+		(at 90.17 207.01)
 	)
 	(no_connect
