File: SmokeSensor/Hardware/LCD.kicad_sch (KiCad schematic)
At the start: 2 parts, among them J3 Conn_01x11, J4 Conn_01x04

Commit message: edit HBridge, RTC_Pump, SmokeSensor skillscreen layers
Parts:
- J3: footprint Connector_PinHeader_2.54mm:PinHeader_1x11_P2.54mm_Vertical -> Connector_PinSocket_2.54mm:PinSocket_1x11_P2.54mm_Vertical
Changed lines of the file:
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@@
 			)
 		)
-		(property "Footprint" "Connector_PinHeader_2.54mm:PinHeader_1x11_P2.54mm_Vertical"
+		(property "Footprint" "Connector_PinSocket_2.54mm:PinSocket_1x11_P2.54mm_Vertical"
 			(at 111.76 115.57 0)
 			(hide yes)
