File: SmokeSensor/Hardware/POWER.kicad_sch (KiCad schematic)
At the start: 21 parts, among them J5 Pin lithium, J6 Switch, U1 MT3608, U2 TP4056-42-ESOP8, U3 MCP1700x-330xxMB

Commit message: edit HBridge, RTC_Pump, SmokeSensor skillscreen layers
Changed lines of the file:
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@@
 		(dnp no)
 		(property "Reference" "L1"
-			(at 112.776 42.418 90)
+			(at 115.57 42.418 90)
 			(show_name no)
 			(do_not_autoplace no)
@@
 		)
 		(property "Value" "22uH/2A"
-			(at 118.11 42.418 90)
+			(at 115.824 45.974 90)
 			(show_name no)
 			(do_not_autoplace no)
