File: SmokeSensor/Hardware/SmokeSensor.kicad_pcb (KiCad board)
At the start: 2 copper layers, 84 x 63 mm, 59 parts, among them J1 USB_C_Receptacle_USB2.0_16P, J2 Conn_01x05_Pin, J3 Conn_01x11, J4 Conn_01x04, J5 Pin lithium, J6 Switch, Q1 SS8050, Q2 SS8050, SW1 RESET, SW2 BOOT, U1 MT3608, U2 TP4056-42-ESOP8, U3 MCP1700x-330xxMB, U4 CH340C, U5 SHT31-DIS, U6 ESP32-WROOM-32E

Commit message: edit HBridge, RTC_Pump, SmokeSensor skillscreen layers
Parts:
- added G***: LOGO, Smoke:img, F.Cu at (186.9, 113.7)
- J3: footprint Connector_PinHeader_2.54mm:PinHeader_1x11_P2.54mm_Vertical -> Connector_PinSocket_2.54mm:PinSocket_1x11_P2.54mm_Vertical
Routing:
- net +3.3V: track 140.1 -> 159.6 mm
- net GND: track 65.9 -> 66.8 mm, vias 345 -> 157
Other:
- board text added: "BOOT"
- board text added: "CHARGE"
- board text added: "LCD TFT"
- board text added: "UART"
- board text removed: "DUC ANH"
- board text removed: "FLASH"
