File: RTC_PUMP12V5A_v2/MCU.kicad_sch (KiCad schematic)
At the start: 25 parts, among them J3 USB_C_Receptacle_USB2.0_16P, SW1 SW_Push, SW2 SW_Push, U2 USBLC6-2SC6, U4 ESP32-C3-WROOM-02, U8 ESP32-S3-WROOM-1

Commit message: finished the layout & routed this circuit
Parts:
- removed C21: 10u, Capacitor_SMD:C_0805_2012Metric, symbol Device:C_Small
- removed R31: 10k, Resistor_SMD:R_0805_2012Metric, symbol Device:R_Small_US
- removed U8: ESP32-S3-WROOM-1, RF_Module:ESP32-S3-WROOM-1, symbol RF_Module:ESP32-S3-WROOM-1
- renumbered C1 to C10, C2 to C11, C11 to C12, C12 to C13, C13 to C14, C14 to C15, D1 to D5, J3 to J2, R9 to R10, R16 to R11, R17 to R12, R12 to R13, R13 to R14, R14 to R7, R15 to R8, R8 to R9, U2 to U3
