File: RTC_PUMP12V5A_v2/Mosfet.kicad_sch (KiCad schematic)
At the start: 23 parts, among them J5 Pump, J6 Pump, Q2 IRLR7843, Q3 IRLR7843, U6 PC817, U7 PC817

Commit message: finished the layout & routed this circuit
Parts:
- C18: renamed from C24; footprint Capacitor_SMD:CP_Elec_8x10.5 -> Capacitor_THT:CP_Radial_D10.0mm_P5.00mm
- C19: renamed from C25; footprint Capacitor_SMD:CP_Elec_8x10.5 -> Capacitor_THT:CP_Radial_D10.0mm_P5.00mm
- C20: renamed from C26; footprint Capacitor_SMD:CP_Elec_8x10.5 -> Capacitor_THT:CP_Radial_D10.0mm_P5.00mm
- D8, D9: footprint Diode_SMD:ST_D_SMC -> TV_ChanSMD:Diode SS54
- renumbered J5 to J3, J6 to J4, R20 to R17, R21 to R18, R23 to R19, R24 to R20, R25 to R21, R26 to R22, R27 to R23, R28 to R24, R29 to R25, R30 to R26
Connections:
- net IO9 renamed IO10
Changed lines of the file:
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@@
 		)
 	)
-	(global_label "IO9"
+	(global_label "IO10"
 		(shape input)
 		(at 99.06 124.46 180)
@@
 		)
 		(property "Intersheetrefs" "${INTERSHEET_REFS}"
-			(at 92.93 124.46 0)
+			(at 91.7205 124.46 0)
 			(hide yes)
 			(show_name no)
@@
 			)
 		)
-		(property "Footprint" "Diode_SMD:ST_D_SMC"
+		(property "Footprint" "TV_ChanSMD:Diode SS54"
 			(at 154.305 114.3 0)
 			(hide yes)
@@
 			)
 		)
-		(property "Footprint" "Diode_SMD:ST_D_SMC"
+		(property "Footprint" "TV_ChanSMD:Diode SS54"
 			(at 155.575 62.23 0)
 			(hide yes)
@@
 		(in_pos_files yes)
 		(dnp no)
-		(property "Reference" "#PWR041"
+		(property "Reference" "#PWR037"
 			(at 151.13 147.32 0)
 			(hide yes)
@@
 			(project "RTC_PUMP12V5A_V2"
 				(path "/18f8a9b7-bab5-436b-ad60-d98bac7a6ef4/7449cd4e-2585-41f8-94cd-f1ee70952816"
-					(reference "#PWR041")
+					(reference "#PWR037")
 					(unit 1)
 				)
@@
 		(in_pos_files yes)
 		(dnp no)
-		(property "Reference" "R29"
+		(property "Reference" "R25"
 			(at 147.828 118.364 0)
 			(show_name no)
@@
 			(project "RTC_PUMP12V5A_V2"
 				(path "/18f8a9b7-bab5-436b-ad60-d98bac7a6ef4/7449cd4e-2585-41f8-94cd-f1ee70952816"
-					(reference "R29")
+					(reference "R25")
 					(unit 1)
 				)
@@
 		(in_pos_files yes)
 		(dnp no)
-		(property "Reference" "R20"
+		(property "Reference" "R17"
 			(at 103.886 119.888 90)
 			(show_name no)
@@
 			(project "RTC_PUMP12V5A_V2"
 				(path "/18f8a9b7-bab5-436b-ad60-d98bac7a6ef4/7449cd4e-2585-41f8-94cd-f1ee70952816"
-					(reference "R20")
+					(reference "R17")
 					(unit 1)
 				)
@@
 		(in_pos_files yes)
 		(dnp no)
-		(property "Reference" "J5"
+		(property "Reference" "J3"
 			(at 173.99 115.5701 0)
 			(show_name no)
@@
 			(project "RTC_PUMP12V5A_V2"
 				(path "/18f8a9b7-bab5-436b-ad60-d98bac7a6ef4/7449cd4e-2585-41f8-94cd-f1ee70952816"
-					(reference "J5")
+					(reference "J3")
 					(unit 1)
 				)
@@
 		(in_pos_files yes)
 		(dnp no)
-		(property "Reference" "R25"
+		(property "Reference" "R21"
 			(at 135.89 124.714 90)
 			(show_name no)
@@
 			(project "RTC_PUMP12V5A_V2"
 				(path "/18f8a9b7-bab5-436b-ad60-d98bac7a6ef4/7449cd4e-2585-41f8-94cd-f1ee70952816"
-					(reference "R25")
+					(reference "R21")
 					(unit 1)
 				)
@@
 		(in_pos_files yes)
 		(dnp no)
-		(property "Reference" "R24"
+		(property "Reference" "R20"
 			(at 128.778 61.214 0)
 			(show_name no)
@@
 			(project "RTC_PUMP12V5A_V2"
 				(path "/18f8a9b7-bab5-436b-ad60-d98bac7a6ef4/7449cd4e-2585-41f8-94cd-f1ee70952816"
-					(reference "R24")
+					(reference "R20")
 					(unit 1)
 				)
@@
 		(in_pos_files yes)
 		(dnp no)
-		(property "Reference" "R21"
+		(property "Reference" "R18"
 			(at 105.156 67.818 90)
 			(show_name no)
@@
 			(project "RTC_PUMP12V5A_V2"
 				(path "/18f8a9b7-bab5-436b-ad60-d98bac7a6ef4/7449cd4e-2585-41f8-94cd-f1ee70952816"
-					(reference "R21")
+					(reference "R18")
 					(unit 1)
 				)
@@
 		(in_pos_files yes)
 		(dnp no)
-		(property "Reference" "R30"
+		(property "Reference" "R26"
 			(at 149.098 66.294 0)
 			(show_name no)
@@
 			(project "RTC_PUMP12V5A_V2"
 				(path "/18f8a9b7-bab5-436b-ad60-d98bac7a6ef4/7449cd4e-2585-41f8-94cd-f1ee70952816"
-					(reference "R30")
+					(reference "R26")
 					(unit 1)
 				)
@@
 		(in_pos_files yes)
 		(dnp no)
-		(property "Reference" "C26"
+		(property "Reference" "C20"
 			(at 210.312 89.154 0)
 			(show_name no)
@@
 			)
 		)
-		(property "Footprint" "Capacitor_SMD:CP_Elec_8x10.5"
+		(property "Footprint" "Capacitor_THT:CP_Radial_D10.0mm_P5.00mm"
 			(at 208.28 90.17 0)
 			(hide yes)
@@
 			(project "RTC_PUMP12V5A_V2"
 				(path "/18f8a9b7-bab5-436b-ad60-d98bac7a6ef4/7449cd4e-2585-41f8-94cd-f1ee70952816"
-					(reference "C26")
+					(reference "C20")
 					(unit 1)
 				)
@@
 		(in_pos_files yes)
 		(dnp no)
-		(property "Reference" "#PWR049"
+		(property "Reference" "#PWR041"
 			(at 198.12 104.14 0)
 			(hide yes)
@@
 			(project "RTC_PUMP12V5A_V2"
 				(path "/18f8a9b7-bab5-436b-ad60-d98bac7a6ef4/7449cd4e-2585-41f8-94cd-f1ee70952816"
-					(reference "#PWR049")
+					(reference "#PWR041")
 					(unit 1)
 				)
@@
 		(in_pos_files yes)
 		(dnp no)
-		(property "Reference" "R26"
+		(property "Reference" "R22"
 			(at 137.16 72.644 90)
 			(show_name no)
@@
 			(project "RTC_PUMP12V5A_V2"
 				(path "/18f8a9b7-bab5-436b-ad60-d98bac7a6ef4/7449cd4e-2585-41f8-94cd-f1ee70952816"
-					(reference "R26")
+					(reference "R22")
 					(unit 1)
 				)
@@
 		(in_pos_files yes)
 		(dnp no)
-		(property "Reference" "J6"
+		(property "Reference" "J4"
 			(at 175.26 63.5001 0)
 			(show_name no)
@@
 			(project "RTC_PUMP12V5A_V2"
 				(path "/18f8a9b7-bab5-436b-ad60-d98bac7a6ef4/7449cd4e-2585-41f8-94cd-f1ee70952816"
-					(reference "J6")
+					(reference "J4")
 					(unit 1)
 				)
@@
 		(in_pos_files yes)
 		(dnp no)
-		(property "Reference" "C24"
+		(property "Reference" "C18"
 			(at 189.992 89.408 0)
 			(show_name no)
@@
 			)
 		)
-		(property "Footprint" "Capacitor_SMD:CP_Elec_8x10.5"
+		(property "Footprint" "Capacitor_THT:CP_Radial_D10.0mm_P5.00mm"
 			(at 187.96 90.17 0)
 			(hide yes)
@@
 			(project "RTC_PUMP12V5A_V2"
 				(path "/18f8a9b7-bab5-436b-ad60-d98bac7a6ef4/7449cd4e-2585-41f8-94cd-f1ee70952816"
-					(reference "C24")
+					(reference "C18")
 					(unit 1)
 				)
@@
 		(in_pos_files yes)
 		(dnp no)
-		(property "Reference" "C25"
+		(property "Reference" "C19"
 			(at 200.152 89.408 0)
 			(show_name no)
@@
 			)
 		)
-		(property "Footprint" "Capacitor_SMD:CP_Elec_8x10.5"
+		(property "Footprint" "Capacitor_THT:CP_Radial_D10.0mm_P5.00mm"
 			(at 198.12 90.17 0)
 			(hide yes)
@@
 			(project "RTC_PUMP12V5A_V2"
 				(path "/18f8a9b7-bab5-436b-ad60-d98bac7a6ef4/7449cd4e-2585-41f8-94cd-f1ee70952816"
-					(reference "C25")
+					(reference "C19")
 					(unit 1)
 				)
@@
 		(in_pos_files yes)
 		(dnp no)
-		(property "Reference" "#PWR048"
+		(property "Reference" "#PWR040"
 			(at 198.12 85.09 0)
 			(hide yes)
@@
 			(project "RTC_PUMP12V5A_V2"
 				(path "/18f8a9b7-bab5-436b-ad60-d98bac7a6ef4/7449cd4e-2585-41f8-94cd-f1ee70952816"
-					(reference "#PWR048")
+					(reference "#PWR040")
 					(unit 1)
 				)
@@
 		(in_pos_files yes)
 		(dnp no)
-		(property "Reference" "R27"
+		(property "Reference" "R23"
 			(at 142.24 133.604 0)
 			(show_name no)
@@
 			(project "RTC_PUMP12V5A_V2"
 				(path "/18f8a9b7-bab5-436b-ad60-d98bac7a6ef4/7449cd4e-2585-41f8-94cd-f1ee70952816"
-					(reference "R27")
+					(reference "R23")
 					(unit 1)
 				)
@@
 		(in_pos_files yes)
 		(dnp no)
-		(property "Reference" "#PWR043"
+		(property "Reference" "#PWR039"
 			(at 152.4 95.25 0)
 			(hide yes)
@@
 			(project "RTC_PUMP12V5A_V2"
 				(path "/18f8a9b7-bab5-436b-ad60-d98bac7a6ef4/7449cd4e-2585-41f8-94cd-f1ee70952816"
-					(reference "#PWR043")
+					(reference "#PWR039")
 					(unit 1)
 				)
@@
 		(in_pos_files yes)
 		(dnp no)
-		(property "Reference" "R23"
+		(property "Reference" "R19"
 			(at 127.508 113.284 0)
 			(show_name no)
@@
 			(project "RTC_PUMP12V5A_V2"
 				(path "/18f8a9b7-bab5-436b-ad60-d98bac7a6ef4/7449cd4e-2585-41f8-94cd-f1ee70952816"
-					(reference "R23")
+					(reference "R19")
 					(unit 1)
 				)
@@
 		(in_pos_files yes)
 		(dnp no)
-		(property "Reference" "#PWR042"
+		(property "Reference" "#PWR038"
 			(at 152.4 55.88 0)
 			(hide yes)
@@
 			(project "RTC_PUMP12V5A_V2"
 				(path "/18f8a9b7-bab5-436b-ad60-d98bac7a6ef4/7449cd4e-2585-41f8-94cd-f1ee70952816"
-					(reference "#PWR042")
+					(reference "#PWR038")
 					(unit 1)
 				)
@@
 		(in_pos_files yes)
 		(dnp no)
-		(property "Reference" "R28"
+		(property "Reference" "R24"
 			(at 143.51 81.534 0)
 			(show_name no)
@@
 			(project "RTC_PUMP12V5A_V2"
 				(path "/18f8a9b7-bab5-436b-ad60-d98bac7a6ef4/7449cd4e-2585-41f8-94cd-f1ee70952816"
-					(reference "R28")
+					(reference "R24")
 					(unit 1)
 				)
@@
 		(in_pos_files yes)
 		(dnp no)
-		(property "Reference" "#PWR040"
+		(property "Reference" "#PWR036"
 			(at 151.13 107.95 0)
 			(hide yes)
@@
 			(project "RTC_PUMP12V5A_V2"
 				(path "/18f8a9b7-bab5-436b-ad60-d98bac7a6ef4/7449cd4e-2585-41f8-94cd-f1ee70952816"
-					(reference "#PWR040")
-					(unit 1)
-				)
+					(reference "#PWR036")
+					(unit 1)
+				)
