File: RTC_PUMP12V5A_v2/Power.kicad_sch (KiCad schematic)
At the start: 25 parts, among them J1 12VDC_IN, Q1 AO4407A, U3 TPS5430DDA, U5 LM1117MP-3.3

Commit message: finished the layout & routed this circuit
Parts:
- added NT1, NT2, NT3, NT4, NT5: NetTie_2, NetTie:NetTie-2_SMD_Pad2.0mm, symbol Device:NetTie_2
- renumbered C23 to C1, C15 to C2, C16 to C3, C7 to C4, C17 to C5, C18 to C6, C8 to C7, C9 to C8, C10 to C9, D2 to D1, D3 to D2, D5 to D3, R7 to R1, R22 to R2, R18 to R3, R19 to R4, TP2 to TP1, TP1 to TP2, U5 to U1, U3 to U2
Connections:
- net GND: now also NT1.2, NT2.2, NT3.2, NT4.2, NT5.2
- net GND_PWR: now also NT1.1, NT2.1, NT3.1, NT4.1, NT5.1
