File: RTC_PUMP12V5A_v2/RTC_PUMP12V5A_V2.kicad_pcb (KiCad board)
At the start: 2 copper layers, 89 parts, among them J1 12VDC_IN, J2 Conn_01x06_Socket, J3 USB_C_Receptacle_USB2.0_16P, J4 UART, J5 Pump, J6 Pump, J7 OLED SPI, Q1 AO4407A, Q2 IRLR7843, Q3 IRLR7843, SW1 SW_Push, SW2 SW_Push, U1 DS3231M, U2 USBLC6-2SC6, U3 TPS5430DDA, U4 ESP32-C3-WROOM-02, U5 LM1117MP-3.3, U6 PC817, U7 PC817

Commit message: finished the layout & routed this circuit
Parts:
- removed the C1 at (191.2, 65.7)
- removed the C15 at (195.7, 71.7)
- removed the D1 at (184.2, 52.9)
- removed the J3 at (211.9, 50.6)
- removed the R11 at (149.6, 72.1)
- removed the R3 at (229.4, 101.4)
- removed the R4 at (229.4, 104.3)
- removed the R8 at (177.9, 61.0)
- removed the U2 at (207.9, 41.4)
- added C10: 10u, Capacitor_SMD:C_0805_2012Metric, F.Cu at (165.4, 73.7)
- added C11: 100n, Capacitor_SMD:C_0805_2012Metric, F.Cu at (162.8, 73.7)
- added D5: SS34, Diode_SMD:D_SMA, F.Cu at (170.4, 73.7)
- added J6: Conn_01x06_Socket, Connector_PinSocket_2.54mm:PinSocket_1x06_P2.54mm_Vertical, F.Cu at (176.5, 90.4)
- added NT1: NetTie_2, NetTie:NetTie-2_SMD_Pad2.0mm, B.Cu at (123.1, 85.1)
- added NT2: NetTie_2, NetTie:NetTie-2_SMD_Pad2.0mm, B.Cu at (123.1, 87.9)
- added NT3: NetTie_2, NetTie:NetTie-2_SMD_Pad2.0mm, B.Cu at (123.1, 90.7)
- added NT4: NetTie_2, NetTie:NetTie-2_SMD_Pad2.0mm, B.Cu at (123.1, 93.4)
- added NT5: NetTie_2, NetTie:NetTie-2_SMD_Pad2.0mm, B.Cu at (123.2, 96.3)
- added R27: 0R, Resistor_SMD:R_0805_2012Metric, F.Cu at (172.6, 82.8)
- added R28: 0R, Resistor_SMD:R_0805_2012Metric, F.Cu at (172.6, 80.3)
- added R29: 0R, Resistor_SMD:R_0805_2012Metric, F.Cu at (172.1, 98.7)
- added R30: 0R, Resistor_SMD:R_0805_2012Metric, F.Cu at (172.1, 101.2)
- added U3: USBLC6-2SC6, PumpTimer:SOT95P280X145-6N, F.Cu at (168.2, 66.4)
- C18: renamed from C24; footprint Capacitor_SMD:CP_Elec_8x10.5 -> Capacitor_THT:CP_Radial_D10.0mm_P5.00mm
- C19: renamed from C25; footprint Capacitor_SMD:CP_Elec_8x10.5 -> Capacitor_THT:CP_Radial_D10.0mm_P5.00mm
- C2: value 100n -> 10u
- C20: renamed from C26; footprint Capacitor_SMD:CP_Elec_8x10.5 -> Capacitor_THT:CP_Radial_D10.0mm_P5.00mm
- D8, D9: footprint Diode_SMD:ST_D_SMC -> TV_ChanSMD:Diode SS54
- J2: value Conn_01x06_Socket -> USB_C_Receptacle_USB2.0_16P; footprint Connector_PinSocket_2.54mm:PinSocket_1x06_P2.54mm_Vertical -> Connector_USB:USB_C_Receptacle_HRO_TYPE-C-31-M-12
- R10: value 0R -> 22
- moved F1 123.8 mm to (114.1, 116.9), turned to 90 degrees
- moved D1 120.2 mm to (126.6, 118.7), turned to 90 degrees
- moved J1 115.8 mm to (109.8, 118.2)
- moved H1 113.9 mm to (105.5, 129.2)
- moved L1 94.2 mm to (162.4, 125.4), turned to 90 degrees
- moved BT1 91.1 mm to (134.4, 99.7)
- moved D2 90.7 mm to (130.0, 127.6), turned to 180 degrees
- moved H2 86.2 mm to (177.5, 129.2)
- moved C1 86.1 mm to (138.2, 119.6)
- moved C9 85.7 mm to (150.8, 115.3), turned to 180 degrees
- moved R1 85.3 mm to (120.0, 120.8), turned to -90 degrees
- moved Q1 83.6 mm to (120.1, 116.1), turned to 180 degrees
- moved D4 81.9 mm to (147.3, 130.6)
- moved C15 79.4 mm to (132.9, 55.8), turned to 90 degrees
- moved D3 79.1 mm to (179.5, 112.5), turned to 90 degrees
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- renumbered TP2 to 3V3, TP1 to 5V, C23 to C1, C11 to C12, C12 to C13, C13 to C14, C14 to C15, C3 to C16, C4 to C17, C19 to C21, C20 to C22, C16 to C3, C7 to C4, C17 to C5, C18 to C6, C8 to C7, C9 to C8, C10 to C9, D2 to D1, D3 to D2, D5 to D3, J5 to J3, J6 to J4, J4 to J5, R7 to R1, R16 to R11, R17 to R12, R12 to R13, R13 to R14, R1 to R15, R2 to R16, R20 to R17, R21 to R18, R23 to R19, R22 to R2, R24 to R20, R25 to R21, R26 to R22, R27 to R23, R28 to R24, R29 to R25, R30 to R26, R18 to R3, R19 to R4, R14 to R7, R15 to R8, U5 to U1, U3 to U2, U1 to U5
Connections:
- J1 pad 3: (no net) -> GND_PWR
- J5 pad 2: Net-(J4-Pin_2) -> Net-(J5-Pin_2)
- J7 pad 5: IO3 -> IO5
- J7 pad 6: IO5 -> IO4
- J7 pad 7: IO4 -> IO3
- R10 pad 1: IO21 -> Net-(R10-Pad1)
- R10 pad 2: Net-(J4-Pin_2) -> USB_D+
- R17 pad 1: IO19 -> IO10
- R5 pad 1: Net-(J3-CC1) -> Net-(J2-CC1)
- R6 pad 1: Net-(J3-CC2) -> Net-(J2-CC2)
- R9 pad 2: USB_D+ -> USB_D-
- U5 pad 14: Net-(U1-VBAT) -> Net-(U5-VBAT)
Routing:
- net IO20: track 0.00 -> 80.0 mm, vias 0 -> 2
- net IO1: track 0.00 -> 64.4 mm, vias 0 -> 3
- net IO10: track 0.00 -> 61.9 mm, vias 0 -> 2
- net IO0: track 0.00 -> 60.4 mm, vias 0 -> 2
- net 5V: track 0.00 -> 41.8 mm
- net Net-(U5-VBAT): track 0.00 -> 37.6 mm
- net IO4: track 0.00 -> 33.4 mm, vias 0 -> 1
- net GND: track 0.00 -> 31.5 mm, vias 0 -> 36
- net EN: track 0.00 -> 30.6 mm
- net IO5: track 0.00 -> 30.5 mm, vias 0 -> 1
- net IO21: track 0.00 -> 28.7 mm
- net IO6: track 0.00 -> 27.8 mm
- net IO7: track 0.00 -> 26.4 mm, vias 0 -> 1
- net IO3: track 0.00 -> 25.3 mm, vias 0 -> 1
- net VIN: track 0.00 -> 17.2 mm
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- added copper zone on F.Cu, net +3.3V
- added copper zone on F.Cu, net 5V
- added copper zone on B.Cu, net GND
- added copper zone on B.Cu, net GND_PWR
- added copper zone on F.Cu, net VIN
Other:
- board outline added: 80 x 80 mm
- board text added: "3V3"
- board text added: "BAT"
- board text added: "BOOT"
- board text added: "GND"
- board text added: "OLED"
- board text added: "OUT1"
- board text added: "OUT2"
- board text added: "RESET"
- board text added: "SCL"
- board text added: "SDA"
- board text added: "USB"
- board text added: "VIN"
