File: RTC_PUMP12V5A_v2/Sensor.kicad_sch (KiCad schematic)
At the start: 6 parts, among them U1 DS3231M

Commit message: finished the layout & routed this circuit
Parts:
- renumbered C3 to C16, C4 to C17, R1 to R15, R2 to R16, U1 to U5
Changed lines of the file:
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@@
 		(in_pos_files yes)
 		(dnp no)
-		(property "Reference" "#PWR04"
+		(property "Reference" "#PWR031"
 			(at 149.86 121.92 0)
 			(hide yes)
@@
 			(project "RTC_PUMP12V5A_V2"
 				(path "/18f8a9b7-bab5-436b-ad60-d98bac7a6ef4/e5dddaf9-ba61-45d8-8028-21653b864f07"
-					(reference "#PWR04")
+					(reference "#PWR031")
 					(unit 1)
 				)
@@
 		(in_pos_files yes)
 		(dnp no)
-		(property "Reference" "#PWR012"
+		(property "Reference" "#PWR032"
 			(at 177.8 77.47 0)
 			(hide yes)
@@
 			(project "RTC_PUMP12V5A_V2"
 				(path "/18f8a9b7-bab5-436b-ad60-d98bac7a6ef4/e5dddaf9-ba61-45d8-8028-21653b864f07"
-					(reference "#PWR012")
+					(reference "#PWR032")
 					(unit 1)
 				)
@@
 		(in_pos_files yes)
 		(dnp no)
-		(property "Reference" "#PWR03"
+		(property "Reference" "#PWR030"
 			(at 147.32 90.17 0)
 			(hide yes)
@@
 			(project "RTC_PUMP12V5A_V2"
 				(path "/18f8a9b7-bab5-436b-ad60-d98bac7a6ef4/e5dddaf9-ba61-45d8-8028-21653b864f07"
-					(reference "#PWR03")
+					(reference "#PWR030")
 					(unit 1)
 				)
@@
 		(in_pos_files yes)
 		(dnp no)
-		(property "Reference" "C3"
+		(property "Reference" "C16"
 			(at 168.91 78.232 0)
 			(show_name no)
@@
 			(project "RTC_PUMP12V5A_V2"
 				(path "/18f8a9b7-bab5-436b-ad60-d98bac7a6ef4/e5dddaf9-ba61-45d8-8028-21653b864f07"
-					(reference "C3")
+					(reference "C16")
 					(unit 1)
 				)
@@
 		(dnp no)
 		(fields_autoplaced yes)
-		(property "Reference" "#FLG01"
+		(property "Reference" "#FLG02"
 			(at 156.21 88.265 0)
 			(hide yes)
@@
 			(project "RTC_PUMP12V5A_V2"
 				(path "/18f8a9b7-bab5-436b-ad60-d98bac7a6ef4/e5dddaf9-ba61-45d8-8028-21653b864f07"
-					(reference "#FLG01")
+					(reference "#FLG02")
 					(unit 1)
 				)
@@
 		(in_pos_files yes)
 		(dnp no)
-		(property "Reference" "#PWR013"
+		(property "Reference" "#PWR033"
 			(at 177.8 90.17 0)
 			(hide yes)
@@
 			(project "RTC_PUMP12V5A_V2"
 				(path "/18f8a9b7-bab5-436b-ad60-d98bac7a6ef4/e5dddaf9-ba61-45d8-8028-21653b864f07"
-					(reference "#PWR013")
+					(reference "#PWR033")
 					(unit 1)
 				)
@@
 		(dnp no)
 		(fields_autoplaced yes)
-		(property "Reference" "#PWR01"
+		(property "Reference" "#PWR029"
 			(at 128.27 90.17 0)
 			(hide yes)
@@
 			(project "RTC_PUMP12V5A_V2"
 				(path "/18f8a9b7-bab5-436b-ad60-d98bac7a6ef4/e5dddaf9-ba61-45d8-8028-21653b864f07"
-					(reference "#PWR01")
+					(reference "#PWR029")
 					(unit 1)
 				)
@@
 		(in_pos_files yes)
 		(dnp no)
-		(property "Reference" "R1"
+		(property "Reference" "R15"
 			(at 124.46 89.916 0)
 			(show_name no)
@@
 			(project "RTC_PUMP12V5A_V2"
 				(path "/18f8a9b7-bab5-436b-ad60-d98bac7a6ef4/e5dddaf9-ba61-45d8-8028-21653b864f07"
-					(reference "R1")
+					(reference "R15")
 					(unit 1)
 				)
@@
 		(in_pos_files yes)
 		(dnp no)
-		(property "Reference" "R2"
+		(property "Reference" "R16"
 			(at 132.334 89.916 0)
 			(show_name no)
@@
 			(project "RTC_PUMP12V5A_V2"
 				(path "/18f8a9b7-bab5-436b-ad60-d98bac7a6ef4/e5dddaf9-ba61-45d8-8028-21653b864f07"
-					(reference "R2")
+					(reference "R16")
 					(unit 1)
 				)
@@
 		(dnp no)
 		(fields_autoplaced yes)
-		(property "Reference" "U1"
+		(property "Reference" "U5"
 			(at 152.0033 113.03 0)
 			(show_name no)
@@
 			(project "RTC_PUMP12V5A_V2"
 				(path "/18f8a9b7-bab5-436b-ad60-d98bac7a6ef4/e5dddaf9-ba61-45d8-8028-21653b864f07"
-					(reference "U1")
+					(reference "U5")
 					(unit 1)
 				)
@@
 		(in_pos_files yes)
 		(dnp no)
-		(property "Reference" "C4"
+		(property "Reference" "C17"
 			(at 186.69 79.248 0)
 			(show_name no)
@@
 			(project "RTC_PUMP12V5A_V2"
 				(path "/18f8a9b7-bab5-436b-ad60-d98bac7a6ef4/e5dddaf9-ba61-45d8-8028-21653b864f07"
-					(reference "C4")
-					(unit 1)
-				)
+					(reference "C17")
+					(unit 1)
+				)
