File: RTC_PUMP12V5A_v2/peripherals.kicad_sch (KiCad schematic)
At the start: 13 parts, among them J2 Conn_01x06_Socket, J4 UART, J7 OLED SPI

Commit message: finished the layout & routed this circuit
Parts:
- renumbered C19 to C21, C20 to C22, J4 to J5, J2 to J6, R10 to R27, R11 to R28, R3 to R29, R4 to R30
Connections:
- net IO0: now also R29.1; no longer R30.1
- net IO1: now also R30.1; no longer R29.1
- net IO20: now also R27.1; no longer R28.1
- net IO21: now also R28.1; no longer R27.1
- net IO3: now also J7.7 (Pin_7); no longer J7.5 (Pin_5)
- net IO4: now also J7.6 (Pin_6); no longer J7.7 (Pin_7)
- net IO5: now also J7.5 (Pin_5); no longer J7.6 (Pin_6)
Changed lines of the file:
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@@
 	(text "TXD"
 		(exclude_from_sim no)
-		(at 99.06 90.424 0)
+		(at 100.838 92.964 0)
 		(effects
 			(font
@@
 	(text "RXD\n"
 		(exclude_from_sim no)
-		(at 99.314 92.964 0)
+		(at 100.838 90.424 0)
 		(effects
 			(font
@@
 				)
 			)
-			(table_cell "IO3"
+			(table_cell "IO5\n"
 				(exclude_from_sim no)
 				(at 210.82 69.85 0)
@@
 				)
 			)
-			(table_cell "IO5"
+			(table_cell "IO3"
 				(exclude_from_sim no)
 				(at 210.82 74.93 0)
@@
 	(global_label "IO5"
 		(shape input)
+		(at 207.01 96.52 0)
+		(fields_autoplaced yes)
+		(effects
+			(font
+				(size 1.27 1.27)
+			)
+			(justify left)
+		)
+		(property "Intersheetrefs" "${INTERSHEET_REFS}"
+			(at 213.14 96.52 0)
+			(hide yes)
+			(show_name no)
+			(do_not_autoplace no)
+			(effects
+				(font
+					(size 1.27 1.27)
+				)
+				(justify left)
+			)
+		)
+	)
+	(global_label "IO4"
+		(shape input)
 		(at 207.01 99.06 0)
 		(fields_autoplaced yes)
@@
 	(global_label "IO0"
 		(shape input)
+		(at 199.39 125.73 0)
+		(fields_autoplaced yes)
+		(effects
+			(font
+				(size 1.27 1.27)
+			)
+			(justify left)
+		)
+		(property "Intersheetrefs" "${INTERSHEET_REFS}"
+			(at 205.52 125.73 0)
+			(hide yes)
+			(show_name no)
+			(do_not_autoplace no)
+			(effects
+				(font
+					(size 1.27 1.27)
+				)
+				(justify left)
+			)
+		)
+	)
+	(global_label "IO1"
+		(shape input)
 		(at 199.39 129.54 0)
 		(fields_autoplaced yes)
@@
 		)
 	)
-	(global_label "IO4"
+	(global_label "IO3"
 		(shape input)
 		(at 207.01 101.6 0)
@@
 		(property "Intersheetrefs" "${INTERSHEET_REFS}"
 			(at 213.14 101.6 0)
-			(hide yes)
-			(show_name no)
-			(do_not_autoplace no)
-			(effects
-				(font
-					(size 1.27 1.27)
-				)
-				(justify left)
-			)
-		)
-	)
-	(global_label "IO20"
-		(shape input)
-		(at 127 95.25 0)
-		(fields_autoplaced yes)
-		(effects
-			(font
-				(size 1.27 1.27)
-			)
-			(justify left)
-		)
-		(property "Intersheetrefs" "${INTERSHEET_REFS}"
-			(at 134.3395 95.25 0)
 			(hide yes)
 			(show_name no)
@@
 		)
 	)
-	(global_label "IO3"
+	(global_label "IO21"
 		(shape input)
-		(at 207.01 96.52 0)
+		(at 127 95.25 0)
 		(fields_autoplaced yes)
 		(effects
@@
 		)
 		(property "Intersheetrefs" "${INTERSHEET_REFS}"
-			(at 213.14 96.52 0)
+			(at 134.3395 95.25 0)
 			(hide yes)
 			(show_name no)
@@
 		)
 	)
-	(global_label "IO21"
+	(global_label "IO20"
 		(shape input)
 		(at 127 87.63 0)
@@
 		(property "Intersheetrefs" "${INTERSHEET_REFS}"
 			(at 134.3395 87.63 0)
-			(hide yes)
-			(show_name no)
-			(do_not_autoplace no)
-			(effects
-				(font
-					(size 1.27 1.27)
-				)
-				(justify left)
-			)
-		)
-	)
-	(global_label "IO1"
-		(shape input)
-		(at 199.39 125.73 0)
-		(fields_autoplaced yes)
-		(effects
-			(font
-				(size 1.27 1.27)
-			)
-			(justify left)
-		)
-		(property "Intersheetrefs" "${INTERSHEET_REFS}"
-			(at 205.52 125.73 0)
 			(hide yes)
 			(show_name no)
@@
 		(in_pos_files yes)
 		(dnp no)
-		(property "Reference" "#PWR06"
+		(property "Reference" "#PWR048"
 			(at 212.09 140.97 0)
 			(hide yes)
@@
 			(project "RTC_PUMP12V5A_V2"
 				(path "/18f8a9b7-bab5-436b-ad60-d98bac7a6ef4/b53245cb-a163-453a-a7c4-f32098b018b7"
-					(reference "#PWR06")
+					(reference "#PWR048")
 					(unit 1)
 				)
@@
 		(in_pos_files yes)
 		(dnp yes)
-		(property "Reference" "R11"
+		(property "Reference" "R28"
 			(at 120.65 91.44 90)
 			(show_name no)
@@
 			(project "RTC_PUMP12V5A_V2"
 				(path "/18f8a9b7-bab5-436b-ad60-d98bac7a6ef4/b53245cb-a163-453a-a7c4-f32098b018b7"
-					(reference "R11")
+					(reference "R28")
 					(unit 1)
 				)
@@
 		(in_pos_files yes)
 		(dnp no)
-		(property "Reference" "#PWR015"
+		(property "Reference" "#PWR042"
 			(at 113.03 88.9 0)
 			(hide yes)
@@
 			(project "RTC_PUMP12V5A_V2"
 				(path "/18f8a9b7-bab5-436b-ad60-d98bac7a6ef4/b53245cb-a163-453a-a7c4-f32098b018b7"
-					(reference "#PWR015")
+					(reference "#PWR042")
 					(unit 1)
 				)
@@
 		(in_pos_files yes)
 		(dnp no)
-		(property "Reference" "J4"
+		(property "Reference" "J5"
 			(at 103.124 100.838 0)
 			(show_name no)
@@
 			(project "RTC_PUMP12V5A_V2"
 				(path "/18f8a9b7-bab5-436b-ad60-d98bac7a6ef4/b53245cb-a163-453a-a7c4-f32098b018b7"
-					(reference "J4")
+					(reference "J5")
 					(unit 1)
 				)
@@
 		(in_pos_files yes)
 		(dnp no)
-		(property "Reference" "#PWR016"
+		(property "Reference" "#PWR043"
 			(at 113.03 104.14 0)
 			(hide yes)
@@
 			(project "RTC_PUMP12V5A_V2"
 				(path "/18f8a9b7-bab5-436b-ad60-d98bac7a6ef4/b53245cb-a163-453a-a7c4-f32098b018b7"
-					(reference "#PWR016")
+					(reference "#PWR043")
 					(unit 1)
 				)
@@
 		(in_pos_files yes)
 		(dnp no)
-		(property "Reference" "C20"
+		(property "Reference" "C22"
 			(at 181.61 92.202 0)
 			(show_name no)
@@
 			(project "RTC_PUMP12V5A_V2"
 				(path "/18f8a9b7-bab5-436b-ad60-d98bac7a6ef4/b53245cb-a163-453a-a7c4-f32098b018b7"
-					(reference "C20")
+					(reference "C22")
 					(unit 1)
 				)
@@
 		(in_pos_files yes)
 		(dnp no)
-		(property "Reference" "C19"
+		(property "Reference" "C21"
 			(at 163.83 92.202 0)
 			(show_name no)
@@
 			(project "RTC_PUMP12V5A_V2"
 				(path "/18f8a9b7-bab5-436b-ad60-d98bac7a6ef4/b53245cb-a163-453a-a7c4-f32098b018b7"
-					(reference "C19")
+					(reference "C21")
 					(unit 1)
 				)
@@
 		(in_pos_files yes)
 		(dnp no)
-		(property "Reference" "J2"
+		(property "Reference" "J6"
 			(at 172.72 128.27 0)
 			(show_name no)
@@
 			(project "RTC_PUMP12V5A_V2"
 				(path "/18f8a9b7-bab5-436b-ad60-d98bac7a6ef4/b53245cb-a163-453a-a7c4-f32098b018b7"
-					(reference "J2")
+					(reference "J6")
 					(unit 1)
 				)
@@
 		(in_pos_files yes)
 		(dnp no)
-		(property "Reference" "#PWR07"
+		(property "Reference" "#PWR049"
 			(at 212.09 147.32 0)
 			(hide yes)
@@
 			(project "RTC_PUMP12V5A_V2"
 				(path "/18f8a9b7-bab5-436b-ad60-d98bac7a6ef4/b53245cb-a163-453a-a7c4-f32098b018b7"
-					(reference "#PWR07")
+					(reference "#PWR049")
 					(unit 1)
 				)
@@
 		(in_pos_files yes)
 		(dnp yes)
-		(property "Reference" "R10"
+		(property "Reference" "R27"
 			(at 120.65 83.82 90)
 			(show_name no)
@@
 			(project "RTC_PUMP12V5A_V2"
 				(path "/18f8a9b7-bab5-436b-ad60-d98bac7a6ef4/b53245cb-a163-453a-a7c4-f32098b018b7"
-					(reference "R10")
+					(reference "R27")
 					(unit 1)
 				)
@@
 		(in_pos_files yes)
 		(dnp yes)
-		(property "Reference" "R4"
+		(property "Reference" "R30"
 			(at 190.5 131.826 90)
 			(show_name no)
@@
 			(project "RTC_PUMP12V5A_V2"
 				(path "/18f8a9b7-bab5-436b-ad60-d98bac7a6ef4/b53245cb-a163-453a-a7c4-f32098b018b7"
-					(reference "R4")
+					(reference "R30")
 					(unit 1)
 				)
@@
 		(in_pos_files yes)
 		(dnp yes)
-		(property "Reference" "R3"
+		(property "Reference" "R29"
 			(at 190.5 121.92 90)
 			(show_name no)
@@
 			(project "RTC_PUMP12V5A_V2"
 				(path "/18f8a9b7-bab5-436b-ad60-d98bac7a6ef4/b53245cb-a163-453a-a7c4-f32098b018b7"
-					(reference "R3")
+					(reference "R29")
 					(unit 1)
 				)
